Commit message: latest pushes

File: humanoid_robot_description/urdf/gazebo_harness.xacro (robot description, xacro)
@@ -1,4 +1,4 @@
 <?xml version="1.0" ?>
-<robot xmlns:xacro="http://www.ros.org/wiki/xacro" name="robotis_humanoid_robot">
+<robot xmlns:xacro="http://www.ros.org/wiki/xacro" name="humanoid_robot">
   <xacro:macro name="add_sim_harness" params="harnessed_link">
     <gazebo>

File: humanoid_robot_description/urdf/humanoid_robot.gazebo.xacro (robot description, xacro)
@@ -3,5 +3,5 @@
   <gazebo>
     <plugin name="gazebo_ros_control" filename="libgazebo_ros_control.so">
-      <robotNamespace>/robotis_humanoid_robot</robotNamespace>
+      <robotNamespace>/humanoid_robot</robotNamespace>
     </plugin>
   </gazebo>
@@ -247,5 +247,5 @@
         <alwaysOn>true</alwaysOn>
         <updateRate>30</updateRate>
-        <cameraName>robotis_humanoid_robot/camera</cameraName>
+        <cameraName>humanoid_robot/camera</cameraName>
         <imageTopicName>image_raw</imageTopicName>
         <cameraInfoTopicName>camera_info</cameraInfoTopicName>
@@ -269,5 +269,5 @@
       <topic>__default_topic__</topic>
       <plugin filename="libgazebo_ros_imu_sensor.so" name="imu_plugin">
-        <topicName>robotis_humanoid_robot/imu</topicName>
+        <topicName>humanoid_robot/imu</topicName>
         <bodyName>body_link</bodyName>
         <updateRateHZ>10.0</updateRateHZ>

File: humanoid_robot_description/urdf/humanoid_robot.structure.head.xacro (robot description, xacro)
@@ -5,5 +5,5 @@
   -->
   <!-- head -->
-  <xacro:macro name="robotis_humanoid_robot_head" params="parent">
+  <xacro:macro name="humanoid_robot_head" params="parent">
   <!-- head yaw joint -->
   <joint name="head_pan" type="revolute">

File: humanoid_robot_description/urdf/humanoid_robot.structure.larm.xacro (robot description, xacro)
@@ -5,5 +5,5 @@
   -->
   <!-- left leg -->
-  <xacro:macro name="robotis_humanoid_robot_l_arm" params="parent">
+  <xacro:macro name="humanoid_robot_l_arm" params="parent">
   <!-- left shoulder pitch joint -->
   <joint name="l_sho_pitch" type="revolute">

File: humanoid_robot_description/urdf/humanoid_robot.structure.lleg.xacro (robot description, xacro)
@@ -5,5 +5,5 @@
   -->
   <!-- left leg -->
-  <xacro:macro name="robotis_humanoid_robot_l_leg" params="parent">
+  <xacro:macro name="humanoid_robot_l_leg" params="parent">
   <!-- left hip yaw joint -->
   <joint name="l_hip_yaw" type="revolute">

File: humanoid_robot_description/urdf/humanoid_robot.structure.rarm.xacro (robot description, xacro)
@@ -5,5 +5,5 @@
   -->
   <!-- right arm -->
-  <xacro:macro name="robotis_humanoid_robot_r_arm" params="parent">
+  <xacro:macro name="humanoid_robot_r_arm" params="parent">
   <!-- right shoulder pitch joint -->
   <joint name="r_sho_pitch" type="revolute">

File: humanoid_robot_description/urdf/humanoid_robot.structure.rleg.xacro (robot description, xacro)
@@ -5,5 +5,5 @@
   -->
   <!-- right leg -->
-  <xacro:macro name="robotis_humanoid_robot_r_leg" params="parent">
+  <xacro:macro name="humanoid_robot_r_leg" params="parent">
   <!-- right hip yaw joint -->
   <joint name="r_hip_yaw" type="revolute">
